File: hardware/left-0.1/cuddly-chainsaw.sch (KiCad schematic (older format))
At the start: 78 parts, among them J1 USB_C_Receptacle_USB2.0, J2 USB_C_Receptacle_USB2.0, SW1 Encoder_MX_RGB, SW10 MX_RGB, SW11 MX_RGB, SW12 MX_RGB, SW13 MX_RGB, SW14 MX_RGB, SW15 MX_RGB, SW16 MX_RGB, SW17 MX_RGB, SW18 MX_RGB, SW19 MX_RGB, SW2 MX_RGB, SW20 MX_RGB, SW21 MX_RGB, SW22 MX_RGB, SW23 MX_RGB, SW24 MX_RGB, SW25 MX_RGB, SW26 MX_RGB, SW27 MX_RGB, SW28 MX_RGB, SW29 MX_RGB, SW3 MX_RGB, SW30 MX_RGB, SW31 MX_RGB, SW32 MX_RGB, SW33 MX_RGB, SW34 MX_RGB, SW4 MX_RGB, SW5 MX_RGB, SW6 MX_RGB, SW7 MX_RGB, SW8 MX_RGB, SW9 MX_RGB, U1 USBLC6-2P6

Commit message: both halves in pcbnew
Parts:
- BZ1: Digikey (none) -> 490-9647-1-ND; LCSC (none) -> NA; MPN (none) -> PKMCS0909E4000
- D1, D10, D12, D13, D14, D15, D16, D17, D18, D19, D2, D20, D21, D22, D23, D24, D25, D26, D27, D28, D29, D3, D30, D31, D32, D33, D34, D35, D4, D5, D6, D7, D8, D9: Digikey (none) -> 1N4148W-FDICT-ND; LCSC (none) -> C83528; MPN (none) -> 1N4148W-7-F
- D11: Digikey (none) -> SDM1100S1F-7DICT-ND; LCSC (none) -> C122853; MPN (none) -> B5817WL
- F1: Digikey (none) -> 507-1813-1-ND; LCSC (none) -> C181350; MPN (none) -> 0ZCK0050FF2E
- J1, J2: Digikey (none) -> NA; LCSC (none) -> C319148; MPN (none) -> U262-161N-4BVC11
- R1, R2: Digikey (none) -> 118-CR0603-JW-512ELFCT-ND; MPN (none) -> CR0603-JW-512ELF
- SW1: footprint (none) -> josh-buttons-switches:MX_KEYSWITCH_ENCODER_RGB; DNP (none) -> DNP; Digikey (none) -> 987-1398-ND; LCSC (none) -> C361165; MPN (none) -> EC11E1834403
- SW10, SW11, SW12, SW13, SW14, SW15, SW16, SW17, SW18, SW19, SW2, SW20, SW21, SW22, SW23, SW24, SW25, SW26, SW27, SW28, SW29, SW3, SW30, SW31, SW32, SW33, SW34, SW4, SW5, SW6, SW7, SW8, SW9: footprint (none) -> josh-buttons-switches:MX_KEYSWITCH_RGB; DNP (none) -> DNP
- U1: value USBLC6-2P6 -> USBLC6-2SC6; Digikey (none) -> 497-5235-1-ND; LCSC (none) -> C7519; MPN (none) -> USBLC6-2SC6

Commit message: first go at board outline done
Parts:
- SW10, SW15, SW20: footprint josh-buttons-switches:MX_KEYSWITCH_RGB -> josh-buttons-switches:MX_KEYSWITCH_RGB_1.25U
- SW25: footprint josh-buttons-switches:MX_KEYSWITCH_RGB -> josh-buttons-switches:MX_KEYSWITCH_RGB_2.75U
- SW7: footprint josh-buttons-switches:MX_KEYSWITCH_RGB -> josh-buttons-switches:MX_KEYSWITCH_RGB_1.5U
- SW8: footprint josh-buttons-switches:MX_KEYSWITCH_RGB -> josh-buttons-switches:MX_KEYSWITCH_RGB_1.75U
- SW9: footprint josh-buttons-switches:MX_KEYSWITCH_RGB -> josh-buttons-switches:MX_KEYSWITCH_RGB_2.25U
Changed lines of the file:
@@
 F 0 "SW7" H 3000 5150 50  0000 C CNN
 F 1 "MX_RGB" H 3100 4600 50  0000 C CNN
-F 2 "josh-buttons-switches:MX_KEYSWITCH_RGB" H 3100 4900 50  0001 C CNN
+F 2 "josh-buttons-switches:MX_KEYSWITCH_RGB_1.5U" H 3100 4900 50  0001 C CNN
 F 3 "~" H 3100 4900 50  0001 C CNN
 F 4 "DNP" H 3100 4700 50  0001 C CNN "DNP"
@@
 F 0 "SW8" H 3050 5900 50  0000 C CNN
 F 1 "MX_RGB" H 3100 5350 50  0000 C CNN
-F 2 "josh-buttons-switches:MX_KEYSWITCH_RGB" H 3100 5650 50  0001 C CNN
+F 2 "josh-buttons-switches:MX_KEYSWITCH_RGB_1.75U" H 3100 5650 50  0001 C CNN
 F 3 "~" H 3100 5650 50  0001 C CNN
 F 4 "DNP" H 3100 5450 50  0001 C CNN "DNP"
@@
 F 0 "SW9" H 3050 6650 50  0000 C CNN
 F 1 "MX_RGB" H 3100 6100 50  0000 C CNN
-F 2 "josh-buttons-switches:MX_KEYSWITCH_RGB" H 3100 6400 50  0001 C CNN
+F 2 "josh-buttons-switches:MX_KEYSWITCH_RGB_2.25U" H 3100 6400 50  0001 C CNN
 F 3 "~" H 3100 6400 50  0001 C CNN
 F 4 "DNP" H 3100 6200 50  0001 C CNN "DNP"
@@
 F 0 "SW10" H 3050 7400 50  0000 C CNN
 F 1 "MX_RGB" H 3100 6850 50  0000 C CNN
-F 2 "josh-buttons-switches:MX_KEYSWITCH_RGB" H 3100 7150 50  0001 C CNN
+F 2 "josh-buttons-switches:MX_KEYSWITCH_RGB_1.25U" H 3100 7150 50  0001 C CNN
 F 3 "~" H 3100 7150 50  0001 C CNN
 F 4 "DNP" H 3100 6950 50  0001 C CNN "DNP"
@@
 F 0 "SW15" H 4150 7400 50  0000 C CNN
 F 1 "MX_RGB" H 4200 6850 50  0000 C CNN
-F 2 "josh-buttons-switches:MX_KEYSWITCH_RGB" H 4200 7150 50  0001 C CNN
+F 2 "josh-buttons-switches:MX_KEYSWITCH_RGB_1.25U" H 4200 7150 50  0001 C CNN
 F 3 "~" H 4200 7150 50  0001 C CNN
 F 4 "DNP" H 4200 6950 50  0001 C CNN "DNP"
@@
 F 0 "SW20" H 5250 7400 50  0000 C CNN
 F 1 "MX_RGB" H 5300 6850 50  0000 C CNN
-F 2 "josh-buttons-switches:MX_KEYSWITCH_RGB" H 5300 7150 50  0001 C CNN
+F 2 "josh-buttons-switches:MX_KEYSWITCH_RGB_1.25U" H 5300 7150 50  0001 C CNN
 F 3 "~" H 5300 7150 50  0001 C CNN
 F 4 "DNP" H 5300 6950 50  0001 C CNN "DNP"
@@
 F 0 "SW25" H 6350 7400 50  0000 C CNN
 F 1 "MX_RGB" H 6400 6850 50  0000 C CNN
-F 2 "josh-buttons-switches:MX_KEYSWITCH_RGB" H 6400 7150 50  0001 C CNN
+F 2 "josh-buttons-switches:MX_KEYSWITCH_RGB_2.75U" H 6400 7150 50  0001 C CNN
 F 3 "~" H 6400 7150 50  0001 C CNN
 F 4 "DNP" H 6400 6950 50  0001 C CNN "DNP"

Commit message: left all connected
Parts:
- added R9: 22R, Resistor_SMD:R_0603_1608Metric, symbol Device:R
- SW25: footprint josh-buttons-switches:MX_KEYSWITCH_RGB_2.75U -> josh-buttons-switches:MX_KEYSWITCH_RGB_2.75U_REV_STABS
Connections:
- net +5V: now also D11.1 (K)
- net GND: now also J1.A1 (GND), J1.A12 (GND), J1.B1 (GND), J1.B12 (GND), J1.S1 (SHIELD)
- net PIEZO: now also R9.2; no longer BZ1.1 (-)
- net LED_DAT renamed LED_KEYS
- new net: BZ1.1 (-), R9.1
Other:
- note added: "Underglow"
Changed lines of the file:
@@
 $Descr A4 11693 8268
 encoding utf-8
-Sheet 1 2
+Sheet 1 3
 Title "LEFT HALF"
 Date "2020-01-09"
@@
 F28 "PF7" B R 6600 2550 50
 $EndSheet
-$Comp
-L Connector:USB_C_Receptacle_USB2.0 J?
-U 1 1 5E18980C
-P 1050 2050
-AR Path="/5E16A0F8/5E18980C" Ref="J?"  Part="1"
-AR Path="/5E18980C" Ref="J1"  Part="1"
-F 0 "J1" H 700 2900 50  0000 C CNN
-F 1 "USB_C_Receptacle_USB2.0" H 1157 2826 50  0000 C CNN
-F 2 "josh-connectors:USB_C_U262-161N-4BVC11" H 1200 2050 50  0001 C CNN
-F 3 "https://www.usb.org/sites/default/files/documents/usb_type-c.zip" H 1200 2050 50  0001 C CNN
-F 4 "NA" H 1050 2050 50  0001 C CNN "Digikey"
-F 5 "C319148" H 1050 2050 50  0001 C CNN "LCSC"
-F 6 "U262-161N-4BVC11" H 1050 2050 50  0001 C CNN "MPN"
-	1    1050 2050
-	1    0    0    -1
-$EndComp
 Wire Wire Line
 	750  2950 750  3000
@@
 L power:GND #PWR?
 U 1 1 5E189814
-P 800 2900
+P 900 3050
 AR Path="/5E16A0F8/5E189814" Ref="#PWR?"  Part="1"
 AR Path="/5E189814" Ref="#PWR0101"  Part="1"
-F 0 "#PWR0101" H 800 2650 50  0001 C CNN
-F 1 "GND" H 805 2727 50  0000 C CNN
-F 2 "" H 800 2900 50  0001 C CNN
-F 3 "" H 800 2900 50  0001 C CNN
-	1    800  2900
+F 0 "#PWR0101" H 900 2800 50  0001 C CNN
+F 1 "GND" H 905 2877 50  0000 C CNN
+F 2 "" H 900 3050 50  0001 C CNN
+F 3 "" H 900 3050 50  0001 C CNN
+	1    900  3050
 	1    0    0    -1
 $EndComp
@@
 $EndComp
 Wire Wire Line
-	4150 1300 4150 1250
+	4250 1450 4250 1400
 Connection ~ 4050 1450
 $Comp
 L power:+5V #PWR?
 U 1 1 5E189852
-P 4150 1250
+P 4250 1400
 AR Path="/5E16A0F8/5E189852" Ref="#PWR?"  Part="1"
 AR Path="/5E189852" Ref="#PWR0104"  Part="1"
-F 0 "#PWR0104" H 4150 1100 50  0001 C CNN
-F 1 "+5V" H 4165 1423 50  0000 C CNN
-F 2 "" H 4150 1250 50  0001 C CNN
-F 3 "" H 4150 1250 50  0001 C CNN
-	1    4150 1250
+F 0 "#PWR0104" H 4250 1250 50  0001 C CNN
+F 1 "+5V" H 4265 1573 50  0000 C CNN
+F 2 "" H 4250 1400 50  0001 C CNN
+F 3 "" H 4250 1400 50  0001 C CNN
+	1    4250 1400
 	1    0    0    -1
 $EndComp
@@
 F 0 "SW25" H 6350 7400 50  0000 C CNN
 F 1 "MX_RGB" H 6400 6850 50  0000 C CNN
-F 2 "josh-buttons-switches:MX_KEYSWITCH_RGB_2.75U" H 6400 7150 50  0001 C CNN
+F 2 "josh-buttons-switches:MX_KEYSWITCH_RGB_2.75U_REV_STABS" H 6400 7150 50  0001 C CNN
 F 3 "~" H 6400 7150 50  0001 C CNN
 F 4 "DNP" H 6400 6950 50  0001 C CNN "DNP"
@@
 Text Notes 4750 3050 0    100  ~ 0
 Key Switch Matrix
-Text Label 4950 900  0    50   ~ 0
+Text Label 5350 1650 0    50   ~ 0
 ROW_1
-Text Label 4950 1000 0    50   ~ 0
+Text Label 5350 1750 0    50   ~ 0
 ROW_2
-Text Label 4950 1100 0    50   ~ 0
+Text Label 7100 2450 2    50   ~ 0
 ROW_3
-Text Label 4950 1200 0    50   ~ 0
+Text Label 7100 2350 2    50   ~ 0
 ROW_4
-Text Label 4950 1300 0    50   ~ 0
+Text Label 5350 2500 0    50   ~ 0
 ROW_5
-Text Label 4950 1450 0    50   ~ 0
+Text Label 7100 2550 2    50   ~ 0
 COL_1
-Text Label 4950 1550 0    50   ~ 0
+Text Label 5350 1950 0    50   ~ 0
 COL_2
-Text Label 4950 1650 0    50   ~ 0
+Text Label 5350 1850 0    50   ~ 0
 COL_3
-Text Label 4950 1750 0    50   ~ 0
+Text Label 5350 2050 0    50   ~ 0
 COL_4
-Text Label 4950 1850 0    50   ~ 0
+Text Label 5350 2400 0    50   ~ 0
 COL_5
-Text Label 4950 1950 0    50   ~ 0
+Text Label 7100 1800 2    50   ~ 0
 COL_6
-Text Label 4950 2050 0    50   ~ 0
+Text Label 7100 1700 2    50   ~ 0
 COL_7
-Text Label 4950 2150 0    50   ~ 0
+Text Label 7100 1500 2    50   ~ 0
 COL_8
 Text Label 5350 1450 0    50   ~ 0
 SCL_SERIAL
-Text Label 4950 2500 0    50   ~ 0
-LED_DAT
-Text Label 4950 2600 0    50   ~ 0
+Text Label 5350 2250 0    50   ~ 0
+LED_KEYS
+Text Label 7100 1900 2    50   ~ 0
 PIEZO
-Text Label 4950 2700 0    50   ~ 0
+Text Label 7100 2250 2    50   ~ 0
 ENC_A
-Text Label 4950 2800 0    50   ~ 0
+Text Label 7100 2150 2    50   ~ 0
 ENC_B
 $Comp
@@
 Text Notes 10250 5700 0    100  ~ 0
 BUZZ BUZZ
-Text Label 10250 5950 0    50   ~ 0
+Text Label 9850 5950 0    50   ~ 0
 PIEZO
-Wire Wire Line
-	10250 5950 10550 5950
 Wire Wire Line
 	1650 3800 1600 3800
@@
 Text Label 1100 3700 0    50   ~ 0
 ENC_A
-Text Label 1100 3600 0    50   ~ 0
-LED_DAT
 Wire Wire Line
 	1100 3600 1650 3600
@@
 Wire Wire Line
 	1600 3500 1650 3500
+$Comp
+L Device:R R9
+U 1 1 5E1D56CD
+P 10350 5950
+F 0 "R9" V 10250 5950 50  0000 C CNN
+F 1 "22R" V 10350 5950 50  0000 C CNN
+F 2 "Resistor_SMD:R_0603_1608Metric" V 10280 5950 50  0001 C CNN
+F 3 "~" H 10350 5950 50  0001 C CNN
+	1    10350 5950
+	0    1    1    0
+$EndComp
+Wire Wire Line
+	9850 5950 10200 5950
+Wire Wire Line
+	10500 5950 10550 5950
+$Sheet
+S 7450 1100 650  200
+U 5E2A8B31
+F0 "LEDs" 100
+F1 "LEDs.sch" 100
+F2 "DIN" I L 7450 1200 50
+$EndSheet
+Text Notes 7450 800  0    100  ~ 0
+Underglow
+Text Label 1100 3600 0    50   ~ 0
+LED_KEYS
+Text Label 7100 2050 2    50   ~ 0
+LED_UNDER
+Text Label 7000 1200 0    50   ~ 0
+LED_UNDER
+Wire Wire Line
+	7000 1200 7450 1200
+$Comp
+L Connector:USB_C_Receptacle_USB2.0 J?
+U 1 1 5E18980C
+P 1050 2050
+AR Path="/5E16A0F8/5E18980C" Ref="J?"  Part="1"
+AR Path="/5E18980C" Ref="J1"  Part="1"
+F 0 "J1" H 700 2900 50  0000 C CNN
+F 1 "USB_C_Receptacle_USB2.0" H 1157 2826 50  0000 C CNN
+F 2 "josh-connectors:USB_C_U262-161N-4BVC11" H 1200 2050 50  0001 C CNN
+F 3 "https://www.usb.org/sites/default/files/documents/usb_type-c.zip" H 1200 2050 50  0001 C CNN
+F 4 "NA" H 1050 2050 50  0001 C CNN "Digikey"
+F 5 "C319148" H 1050 2050 50  0001 C CNN "LCSC"
+F 6 "U262-161N-4BVC11" H 1050 2050 50  0001 C CNN "MPN"
+	1    1050 2050
+	1    0    0    -1
+$EndComp
+Wire Wire Line
+	7100 1900 6600 1900
+Wire Wire Line
+	5350 2250 5850 2250
+Wire Wire Line
+	7100 2050 6600 2050
+Wire Wire Line
+	7100 2250 6600 2250
+Wire Wire Line
+	6600 2150 7100 2150
+Wire Wire Line
+	7100 2550 6600 2550
+Wire Wire Line
+	7100 2450 6600 2450
+Wire Wire Line
+	7100 2350 6600 2350
+Wire Wire Line
+	5350 2500 5850 2500
+Wire Wire Line
+	5350 1650 5850 1650
+Wire Wire Line
+	5350 1750 5850 1750
+Wire Wire Line
+	5350 1950 5850 1950
+Wire Wire Line
+	5350 2400 5850 2400
+Wire Wire Line
+	7100 1800 6600 1800
+Wire Wire Line
+	7100 1700 6600 1700
+Wire Wire Line
+	5350 2050 5850 2050
+Wire Wire Line
+	5350 1850 5850 1850
+Wire Wire Line
+	7100 1500 6600 1500
 $EndSCHEMATC

Commit message: updated components due to jlk change
Parts:
- SW1: footprint josh-buttons-switches:MX_KEYSWITCH_ENCODER_RGB -> josh-keyboard:MX_KEYSWITCH_ENCODER_RGB
- SW10, SW15, SW20: footprint josh-buttons-switches:MX_KEYSWITCH_RGB_1.25U -> josh-keyboard:MX_KEYSWITCH_RGB_1.25U
- SW11, SW12, SW13, SW14, SW16, SW17, SW18, SW19, SW2, SW21, SW22, SW23, SW24, SW26, SW27, SW28, SW29, SW3, SW30, SW31, SW32, SW33, SW34, SW4, SW5, SW6: footprint josh-buttons-switches:MX_KEYSWITCH_RGB -> josh-keyboard:MX_KEYSWITCH_RGB
- SW25: footprint josh-buttons-switches:MX_KEYSWITCH_RGB_2.75U_REV_STABS -> josh-keyboard:MX_KEYSWITCH_RGB_2.75U_REV_STABS
- SW7: footprint josh-buttons-switches:MX_KEYSWITCH_RGB_1.5U -> josh-keyboard:MX_KEYSWITCH_RGB_1.5U
- SW8: footprint josh-buttons-switches:MX_KEYSWITCH_RGB_1.75U -> josh-keyboard:MX_KEYSWITCH_RGB_1.75U
- SW9: footprint josh-buttons-switches:MX_KEYSWITCH_RGB_2.25U -> josh-keyboard:MX_KEYSWITCH_RGB_2.25U

Commit message: more layout
Parts:
- BZ1: DigiKey (none) -> 490-9647-1-ND; Digikey 490-9647-1-ND -> (none)
- D1, D10, D12, D13, D14, D15, D16, D17, D18, D19, D2, D20, D21, D22, D23, D24, D25, D26, D27, D28, D29, D3, D30, D31, D32, D33, D34, D35, D4, D5, D6, D7, D8, D9: DigiKey (none) -> 1N4148W-FDICT-ND; Digikey 1N4148W-FDICT-ND -> (none)
- D11: DigiKey (none) -> SDM1100S1F-7DICT-ND; Digikey SDM1100S1F-7DICT-ND -> (none)
- F1: DigiKey (none) -> 507-1813-1-ND; Digikey 507-1813-1-ND -> (none)
- J1, J2: DigiKey (none) -> NA; Digikey NA -> (none)
- R1, R2: DigiKey (none) -> 118-CR0603-JW-512ELFCT-ND; Digikey 118-CR0603-JW-512ELFCT-ND -> (none)
- SW1: DigiKey (none) -> 987-1398-ND; Digikey 987-1398-ND -> (none)
- U1: DigiKey (none) -> 497-5235-1-ND; Digikey 497-5235-1-ND -> (none)
