File: hardware/right-0.1/32u4-minimal.sch (KiCad schematic (older format))
At the start: 15 parts, among them SW35 SW_Push, U2 ATmega32U4-AU, Y1 16MHz

Commit message: both halves in pcbnew
Parts:
- removed U2: ATmega32U4-AU, Package_QFP:TQFP-44_10x10mm_P0.8mm, symbol MCU_Microchip_ATmega:ATmega32U4-AU
- added U2: ATmega32U4-MU, Package_DFN_QFN:QFN-44-1EP_7x7mm_P0.5mm_EP5.2x5.2mm, symbol MCU_Microchip_ATmega:ATmega32U4-MU
- C1, C2: footprint Capacitor_SMD:C_0402_1005Metric -> Capacitor_SMD:C_0603_1608Metric; Digikey (none) -> 1276-2228-1-ND; MPN (none) -> CL10C220JB8NFNC
- C3, C6, C7: footprint Capacitor_SMD:C_0402_1005Metric -> Capacitor_SMD:C_0603_1608Metric; Digikey (none) -> 1276-1000-1-ND; MPN (none) -> CL10B104KB8NNNC
- C4, C5: footprint Capacitor_SMD:C_0402_1005Metric -> Capacitor_SMD:C_0603_1608Metric; Digikey (none) -> 1276-1866-1-ND; MPN (none) -> CL10A105MP8NNNC
- D36: Digikey (none) -> 732-4980-1-ND; MPN (none) -> 150060VS75000
- R5: Digikey (none) -> CR0603-JW-222ELFCT-ND; MPN (none) -> CR0603-JW-222ELF
- R6: Digikey (none) -> CR0603-JW-103ELFCT-ND; MPN (none) -> CR0603-JW-103ELF
- R7, R8: Digikey (none) -> CR0603-JW-220ELFCT-ND; MPN (none) -> CR0603-JW-220ELF
- SW35: Digikey (none) -> 401-1704-1-ND; LCSC (none) -> C354946; MPN (none) -> KSR223GLFG
- Y1: Digikey (none) -> 535-9134-1-ND; LCSC (none) -> C179641; MPN (none) -> ABM8-16.000MHZ-B2-T
Changed lines of the file:
@@
 F 0 "C7" V 4150 2150 50  0000 C CNN
 F 1 "100n" V 4250 2100 50  0000 C CNN
-F 2 "Capacitor_SMD:C_0402_1005Metric" H 4238 2100 50  0001 C CNN
+F 2 "Capacitor_SMD:C_0603_1608Metric" H 4238 2100 50  0001 C CNN
 F 3 "~" H 4200 2250 50  0001 C CNN
+F 4 "1276-1000-1-ND" H 4200 2250 50  0001 C CNN "Digikey"
+F 5 "CL10B104KB8NNNC" H 4200 2250 50  0001 C CNN "MPN"
 	1    4200 2250
 	0    -1   1    0
@@
 F 0 "C6" V 4150 1900 50  0000 C CNN
 F 1 "100n" V 4250 1850 50  0000 C CNN
-F 2 "Capacitor_SMD:C_0402_1005Metric" H 4238 1850 50  0001 C CNN
+F 2 "Capacitor_SMD:C_0603_1608Metric" H 4238 1850 50  0001 C CNN
 F 3 "~" H 4200 2000 50  0001 C CNN
+F 4 "1276-1000-1-ND" H 4200 2000 50  0001 C CNN "Digikey"
+F 5 "CL10B104KB8NNNC" H 4200 2000 50  0001 C CNN "MPN"
 	1    4200 2000
 	0    -1   1    0
@@
 F 0 "C5" V 4150 1650 50  0000 C CNN
 F 1 "1u" V 4250 1650 50  0000 C CNN
-F 2 "Capacitor_SMD:C_0402_1005Metric" H 4238 1600 50  0001 C CNN
+F 2 "Capacitor_SMD:C_0603_1608Metric" H 4238 1600 50  0001 C CNN
 F 3 "~" H 4200 1750 50  0001 C CNN
+F 4 "1276-1866-1-ND " H 4200 1750 50  0001 C CNN "Digikey"
+F 5 "CL10A105MP8NNNC " H 4200 1750 50  0001 C CNN "MPN"
 	1    4200 1750
 	0    -1   1    0
@@
 F 0 "C1" V 1800 3000 50  0000 C CNN
 F 1 "22p" V 2100 3000 50  0000 C CNN
-F 2 "Capacitor_SMD:C_0402_1005Metric" H 1988 2850 50  0001 C CNN
+F 2 "Capacitor_SMD:C_0603_1608Metric" H 1988 2850 50  0001 C CNN
 F 3 "~" H 1950 3000 50  0001 C CNN
+F 4 "1276-2228-1-ND " H 1950 3000 50  0001 C CNN "Digikey"
+F 5 "CL10C220JB8NFNC " H 1950 3000 50  0001 C CNN "MPN"
 	1    1950 3000
 	0    1    1    0
@@
 F 0 "C2" V 1800 3400 50  0000 C CNN
 F 1 "22p" V 2100 3400 50  0000 C CNN
-F 2 "Capacitor_SMD:C_0402_1005Metric" H 1988 3250 50  0001 C CNN
+F 2 "Capacitor_SMD:C_0603_1608Metric" H 1988 3250 50  0001 C CNN
 F 3 "~" H 1950 3400 50  0001 C CNN
+F 4 "1276-2228-1-ND " H 1950 3400 50  0001 C CNN "Digikey"
+F 5 "CL10C220JB8NFNC " H 1950 3400 50  0001 C CNN "MPN"
 	1    1950 3400
 	0    1    1    0
@@
 F 2 "josh-oscillators:Crystal_SMD_3225-4Pin_3.2x2.5mm" H 2300 3200 50  0001 C CNN
 F 3 "~" H 2300 3200 50  0001 C CNN
+F 4 "535-9134-1-ND" H 2300 3200 50  0001 C CNN "Digikey"
+F 5 "C179641" H 2300 3200 50  0001 C CNN "LCSC"
+F 6 "ABM8-16.000MHZ-B2-T" H 2300 3200 50  0001 C CNN "MPN"
 	1    2300 3200
 	0    1    1    0
@@
 F 0 "C4" H 3215 4446 50  0000 L CNN
 F 1 "1u" H 3215 4355 50  0000 L CNN
-F 2 "Capacitor_SMD:C_0402_1005Metric" H 3138 4250 50  0001 C CNN
+F 2 "Capacitor_SMD:C_0603_1608Metric" H 3138 4250 50  0001 C CNN
 F 3 "~" H 3100 4400 50  0001 C CNN
+F 4 "1276-1866-1-ND " H 3100 4400 50  0001 C CNN "Digikey"
+F 5 "CL10A105MP8NNNC " H 3100 4400 50  0001 C CNN "MPN"
 	1    3100 4400
 	1    0    0    -1
@@
 F 0 "C3" H 2365 3746 50  0000 L CNN
 F 1 "100n" H 2365 3655 50  0000 L CNN
-F 2 "Capacitor_SMD:C_0402_1005Metric" H 2288 3550 50  0001 C CNN
+F 2 "Capacitor_SMD:C_0603_1608Metric" H 2288 3550 50  0001 C CNN
 F 3 "~" H 2250 3700 50  0001 C CNN
+F 4 "1276-1000-1-ND" H 2250 3700 50  0001 C CNN "Digikey"
+F 5 "CL10B104KB8NNNC" H 2250 3700 50  0001 C CNN "MPN"
 	1    2250 3700
 	1    0    0    -1
@@
 F 2 "josh-buttons-switches:BT_Small_2_Pin" H 2450 6100 50  0001 C CNN
 F 3 "~" H 2450 6100 50  0001 C CNN
+F 4 "401-1704-1-ND" H 2450 5900 50  0001 C CNN "Digikey"
+F 5 "C354946" H 2450 5900 50  0001 C CNN "LCSC"
+F 6 "KSR223GLFG" H 2450 5900 50  0001 C CNN "MPN"
 	1    2450 5900
 	1    0    0    -1
@@
 F 2 "Resistor_SMD:R_0603_1608Metric" V 2680 5700 50  0001 C CNN
 F 3 "~" H 2750 5700 50  0001 C CNN
+F 4 "CR0603-JW-103ELFCT-ND  " H 2750 5700 50  0001 C CNN "Digikey"
+F 5 "CR0603-JW-103ELF " H 2750 5700 50  0001 C CNN "MPN"
 	1    2750 5700
 	1    0    0    -1
@@
 F 2 "LED_SMD:LED_0603_1608Metric_Castellated" H 1800 5750 50  0001 C CNN
 F 3 "~" H 1800 5750 50  0001 C CNN
+F 4 "732-4980-1-ND  " H 1800 5750 50  0001 C CNN "Digikey"
+F 5 "150060VS75000" H 1800 5750 50  0001 C CNN "MPN"
 	1    1800 5750
 	0    -1   -1   0
@@
 F 2 "Resistor_SMD:R_0603_1608Metric" V 1730 5400 50  0001 C CNN
 F 3 "~" H 1800 5400 50  0001 C CNN
+F 4 "CR0603-JW-222ELFCT-ND  " H 1800 5400 50  0001 C CNN "Digikey"
+F 5 "CR0603-JW-222ELF " H 1800 5400 50  0001 C CNN "MPN"
 	1    1800 5400
 	1    0    0    -1
@@
 F 2 "Resistor_SMD:R_0603_1608Metric" V 2880 3900 50  0001 C CNN
 F 3 "~" H 2950 3900 50  0001 C CNN
+F 4 "CR0603-JW-220ELFCT-ND  " H 2950 3900 50  0001 C CNN "Digikey"
+F 5 "CR0603-JW-220ELF " H 2950 3900 50  0001 C CNN "MPN"
 	1    2950 3900
 	0    1    1    0
@@
 F 2 "Resistor_SMD:R_0603_1608Metric" V 2880 4000 50  0001 C CNN
 F 3 "~" H 2950 4000 50  0001 C CNN
+F 4 "CR0603-JW-220ELFCT-ND  " H 2950 4000 50  0001 C CNN "Digikey"
+F 5 "CR0603-JW-220ELF " H 2950 4000 50  0001 C CNN "MPN"
 	1    2950 4000
 	0    1    1    0
@@
 PF7
 $Comp
-L MCU_Microchip_ATmega:ATmega32U4-AU U2
-U 1 1 5F4370D6
+L MCU_Microchip_ATmega:ATmega32U4-MU U2
+U 1 1 5FB07BE0
 P 3900 4400
 F 0 "U2" H 3450 6150 50  0000 C CNN
-F 1 "ATmega32U4-AU" V 3900 4400 50  0000 C CNN
-F 2 "Package_QFP:TQFP-44_10x10mm_P0.8mm" H 3900 4400 50  0001 C CIN
+F 1 "ATmega32U4-MU" V 3900 4400 50  0000 C CNN
+F 2 "Package_DFN_QFN:QFN-44-1EP_7x7mm_P0.5mm_EP5.2x5.2mm" H 3900 4400 50  0001 C CIN
 F 3 "http://ww1.microchip.com/downloads/en/DeviceDoc/Atmel-7766-8-bit-AVR-ATmega16U4-32U4_Datasheet.pdf" H 3900 4400 50  0001 C CNN
 	1    3900 4400

Commit message: left all connected
Parts:
- added J3: AVR-ISP-6, josh-connectors:AVR_Programmer_SMD, symbol Connector:AVR-ISP-6
Connections:
- net +5V: now also J3.2 (VCC)
- net GND: now also J3.6 (GND)
- net PB1: now also J3.3 (SCK)
- net PB2: now also J3.4 (MOSI)
- net PB3: now also J3.1 (MISO)
- net nRST: now also J3.5 (~RST)
Other:
- note added: "Programming Header"
Changed lines of the file:
@@
 $Descr A4 11693 8268
 encoding utf-8
-Sheet 2 2
+Sheet 2 3
 Title ""
 Date ""
@@
 	1    0    0    -1
 $EndComp
+$Comp
+L Connector:AVR-ISP-6 J3
+U 1 1 5E3F772B
+P 6450 5550
+F 0 "J3" H 6200 6000 50  0000 R CNN
+F 1 "AVR-ISP-6" H 6800 6000 50  0000 R CNN
+F 2 "josh-connectors:AVR_Programmer_SMD" V 6200 5600 50  0001 C CNN
+F 3 " ~" H 5175 5000 50  0001 C CNN
+	1    6450 5550
+	1    0    0    -1
+$EndComp
+Wire Wire Line
+	6350 5950 6350 6000
+$Comp
+L power:GND #PWR0209
+U 1 1 5E3FABE7
+P 6350 6000
+F 0 "#PWR0209" H 6350 5750 50  0001 C CNN
+F 1 "GND" H 6355 5827 50  0000 C CNN
+F 2 "" H 6350 6000 50  0001 C CNN
+F 3 "" H 6350 6000 50  0001 C CNN
+	1    6350 6000
+	1    0    0    -1
+$EndComp
+Wire Wire Line
+	6350 5050 6350 5000
+$Comp
+L power:+5V #PWR0210
+U 1 1 5E3FD90D
+P 6350 5000
+F 0 "#PWR0210" H 6350 4850 50  0001 C CNN
+F 1 "+5V" H 6365 5173 50  0000 C CNN
+F 2 "" H 6350 5000 50  0001 C CNN
+F 3 "" H 6350 5000 50  0001 C CNN
+	1    6350 5000
+	1    0    0    -1
+$EndComp
+Text Label 7150 5650 2    50   ~ 0
+nRST
+Wire Wire Line
+	7150 5650 6850 5650
+Text Notes 5800 4700 0    100  ~ 0
+Programming Header
+Text HLabel 7150 5350 2    50   BiDi ~ 0
+PB3
+Wire Wire Line
+	7150 5350 6850 5350
+Wire Wire Line
+	6850 5450 7150 5450
+Wire Wire Line
+	6850 5550 7150 5550
+Text HLabel 7150 5550 2    50   BiDi ~ 0
+PB1
+Text HLabel 7150 5450 2    50   BiDi ~ 0
+PB2
 $EndSCHEMATC

Commit message: updated components due to jlk change
Parts:
- J3: footprint josh-connectors:AVR_Programmer_SMD -> josh-connectors:AVR_PROG_2.54_SMT
- SW35: footprint josh-buttons-switches:BT_Small_2_Pin -> josh-buttons-switches:SW_Push_PTS820
Changed lines of the file:
@@
 F 0 "SW35" H 2450 6185 50  0000 C CNN
 F 1 "SW_Push" H 2450 6094 50  0000 C CNN
-F 2 "josh-buttons-switches:BT_Small_2_Pin" H 2450 6100 50  0001 C CNN
+F 2 "josh-buttons-switches:SW_Push_PTS820" H 2450 6100 50  0001 C CNN
 F 3 "~" H 2450 6100 50  0001 C CNN
 F 4 "401-1704-1-ND" H 2450 5900 50  0001 C CNN "Digikey"
@@
 F 0 "J3" H 6200 6000 50  0000 R CNN
 F 1 "AVR-ISP-6" H 6800 6000 50  0000 R CNN
-F 2 "josh-connectors:AVR_Programmer_SMD" V 6200 5600 50  0001 C CNN
+F 2 "josh-connectors:AVR_PROG_2.54_SMT" V 6200 5600 50  0001 C CNN
 F 3 " ~" H 5175 5000 50  0001 C CNN
 	1    6450 5550

Commit message: more layout
Parts:
- C1, C2: DigiKey (none) -> 1276-2228-1-ND; Digikey 1276-2228-1-ND -> (none)
- C3, C6, C7: DigiKey (none) -> 1276-1000-1-ND; Digikey 1276-1000-1-ND -> (none)
- C4, C5: DigiKey (none) -> 1276-1866-1-ND; Digikey 1276-1866-1-ND -> (none)
- D36: DigiKey (none) -> 732-4980-1-ND; Digikey 732-4980-1-ND -> (none)
- R5: DigiKey (none) -> CR0603-JW-222ELFCT-ND; Digikey CR0603-JW-222ELFCT-ND -> (none)
- R6: DigiKey (none) -> CR0603-JW-103ELFCT-ND; Digikey CR0603-JW-103ELFCT-ND -> (none)
- R7, R8: DigiKey (none) -> CR0603-JW-220ELFCT-ND; Digikey CR0603-JW-220ELFCT-ND -> (none)
- SW35: DigiKey (none) -> 401-1704-1-ND; Digikey 401-1704-1-ND -> (none)
- Y1: DigiKey (none) -> 535-9134-1-ND; Digikey 535-9134-1-ND -> (none)
Changed lines of the file:
@@
 F 2 "Capacitor_SMD:C_0603_1608Metric" H 4238 2100 50  0001 C CNN
 F 3 "~" H 4200 2250 50  0001 C CNN
-F 4 "1276-1000-1-ND" H 4200 2250 50  0001 C CNN "Digikey"
+F 4 "1276-1000-1-ND" H 4200 2250 50  0001 C CNN "DigiKey"
 F 5 "CL10B104KB8NNNC" H 4200 2250 50  0001 C CNN "MPN"
 	1    4200 2250
@@
 F 2 "Capacitor_SMD:C_0603_1608Metric" H 4238 1850 50  0001 C CNN
 F 3 "~" H 4200 2000 50  0001 C CNN
-F 4 "1276-1000-1-ND" H 4200 2000 50  0001 C CNN "Digikey"
+F 4 "1276-1000-1-ND" H 4200 2000 50  0001 C CNN "DigiKey"
 F 5 "CL10B104KB8NNNC" H 4200 2000 50  0001 C CNN "MPN"
 	1    4200 2000
@@
 F 2 "Capacitor_SMD:C_0603_1608Metric" H 4238 1600 50  0001 C CNN
 F 3 "~" H 4200 1750 50  0001 C CNN
-F 4 "1276-1866-1-ND " H 4200 1750 50  0001 C CNN "Digikey"
+F 4 "1276-1866-1-ND " H 4200 1750 50  0001 C CNN "DigiKey"
 F 5 "CL10A105MP8NNNC " H 4200 1750 50  0001 C CNN "MPN"
 	1    4200 1750
@@
 F 2 "Capacitor_SMD:C_0603_1608Metric" H 1988 2850 50  0001 C CNN
 F 3 "~" H 1950 3000 50  0001 C CNN
-F 4 "1276-2228-1-ND " H 1950 3000 50  0001 C CNN "Digikey"
+F 4 "1276-2228-1-ND " H 1950 3000 50  0001 C CNN "DigiKey"
 F 5 "CL10C220JB8NFNC " H 1950 3000 50  0001 C CNN "MPN"
 	1    1950 3000
@@
 F 2 "Capacitor_SMD:C_0603_1608Metric" H 1988 3250 50  0001 C CNN
 F 3 "~" H 1950 3400 50  0001 C CNN
-F 4 "1276-2228-1-ND " H 1950 3400 50  0001 C CNN "Digikey"
+F 4 "1276-2228-1-ND " H 1950 3400 50  0001 C CNN "DigiKey"
 F 5 "CL10C220JB8NFNC " H 1950 3400 50  0001 C CNN "MPN"
 	1    1950 3400
@@
 F 2 "josh-oscillators:Crystal_SMD_3225-4Pin_3.2x2.5mm" H 2300 3200 50  0001 C CNN
 F 3 "~" H 2300 3200 50  0001 C CNN
-F 4 "535-9134-1-ND" H 2300 3200 50  0001 C CNN "Digikey"
+F 4 "535-9134-1-ND" H 2300 3200 50  0001 C CNN "DigiKey"
 F 5 "C179641" H 2300 3200 50  0001 C CNN "LCSC"
 F 6 "ABM8-16.000MHZ-B2-T" H 2300 3200 50  0001 C CNN "MPN"
@@
 F 2 "Capacitor_SMD:C_0603_1608Metric" H 3138 4250 50  0001 C CNN
 F 3 "~" H 3100 4400 50  0001 C CNN
-F 4 "1276-1866-1-ND " H 3100 4400 50  0001 C CNN "Digikey"
+F 4 "1276-1866-1-ND " H 3100 4400 50  0001 C CNN "DigiKey"
 F 5 "CL10A105MP8NNNC " H 3100 4400 50  0001 C CNN "MPN"
 	1    3100 4400
@@
 F 2 "Capacitor_SMD:C_0603_1608Metric" H 2288 3550 50  0001 C CNN
 F 3 "~" H 2250 3700 50  0001 C CNN
-F 4 "1276-1000-1-ND" H 2250 3700 50  0001 C CNN "Digikey"
+F 4 "1276-1000-1-ND" H 2250 3700 50  0001 C CNN "DigiKey"
 F 5 "CL10B104KB8NNNC" H 2250 3700 50  0001 C CNN "MPN"
 	1    2250 3700
@@
 F 2 "josh-buttons-switches:SW_Push_PTS820" H 2450 6100 50  0001 C CNN
 F 3 "~" H 2450 6100 50  0001 C CNN
-F 4 "401-1704-1-ND" H 2450 5900 50  0001 C CNN "Digikey"
+F 4 "401-1704-1-ND" H 2450 5900 50  0001 C CNN "DigiKey"
 F 5 "C354946" H 2450 5900 50  0001 C CNN "LCSC"
 F 6 "KSR223GLFG" H 2450 5900 50  0001 C CNN "MPN"
@@
 F 2 "Resistor_SMD:R_0603_1608Metric" V 2680 5700 50  0001 C CNN
 F 3 "~" H 2750 5700 50  0001 C CNN
-F 4 "CR0603-JW-103ELFCT-ND  " H 2750 5700 50  0001 C CNN "Digikey"
+F 4 "CR0603-JW-103ELFCT-ND  " H 2750 5700 50  0001 C CNN "DigiKey"
 F 5 "CR0603-JW-103ELF " H 2750 5700 50  0001 C CNN "MPN"
 	1    2750 5700
@@
 F 2 "LED_SMD:LED_0603_1608Metric_Castellated" H 1800 5750 50  0001 C CNN
 F 3 "~" H 1800 5750 50  0001 C CNN
-F 4 "732-4980-1-ND  " H 1800 5750 50  0001 C CNN "Digikey"
+F 4 "732-4980-1-ND  " H 1800 5750 50  0001 C CNN "DigiKey"
 F 5 "150060VS75000" H 1800 5750 50  0001 C CNN "MPN"
 	1    1800 5750
@@
 F 2 "Resistor_SMD:R_0603_1608Metric" V 1730 5400 50  0001 C CNN
 F 3 "~" H 1800 5400 50  0001 C CNN
-F 4 "CR0603-JW-222ELFCT-ND  " H 1800 5400 50  0001 C CNN "Digikey"
+F 4 "CR0603-JW-222ELFCT-ND  " H 1800 5400 50  0001 C CNN "DigiKey"
 F 5 "CR0603-JW-222ELF " H 1800 5400 50  0001 C CNN "MPN"
 	1    1800 5400
@@
 F 2 "Resistor_SMD:R_0603_1608Metric" V 2880 3900 50  0001 C CNN
 F 3 "~" H 2950 3900 50  0001 C CNN
-F 4 "CR0603-JW-220ELFCT-ND  " H 2950 3900 50  0001 C CNN "Digikey"
+F 4 "CR0603-JW-220ELFCT-ND  " H 2950 3900 50  0001 C CNN "DigiKey"
 F 5 "CR0603-JW-220ELF " H 2950 3900 50  0001 C CNN "MPN"
 	1    2950 3900
@@
 F 2 "Resistor_SMD:R_0603_1608Metric" V 2880 4000 50  0001 C CNN
 F 3 "~" H 2950 4000 50  0001 C CNN
-F 4 "CR0603-JW-220ELFCT-ND  " H 2950 4000 50  0001 C CNN "Digikey"
+F 4 "CR0603-JW-220ELFCT-ND  " H 2950 4000 50  0001 C CNN "DigiKey"
 F 5 "CR0603-JW-220ELF " H 2950 4000 50  0001 C CNN "MPN"
 	1    2950 4000
